Commit message: Refactor code structure and remove redundant code blocks for improved readability and maintainability

File: resource/go2.urdf (robot description, URDF)
Before this commit: robot go2, 23 links, 22 joints
Links:
- link lf_hip_link: geometry collision cylinder length=0.04 radius=0.046; visual mesh filename=package://unitree_go2_description/meshes/hip.dae scale=1 1 1
- link lf_lower_leg_link: geometry collision box size=0.213 0.016 0.016; visual mesh filename=package://unitree_go2_description/meshes/calf.dae scale=1 1 1
- link lf_upper_leg_link: geometry collision box size=0.213 0.0245 0.034; visual mesh filename=package://unitree_go2_description/meshes/thigh.dae scale=1 1 1
- link lh_hip_link: geometry collision cylinder length=0.04 radius=0.046; visual mesh filename=package://unitree_go2_description/meshes/hip.dae scale=1 1 1
- link lh_lower_leg_link: geometry collision box size=0.213 0.016 0.016; visual mesh filename=package://unitree_go2_description/meshes/calf.dae scale=1 1 1
- link lh_upper_leg_link: geometry collision box size=0.213 0.0245 0.034; visual mesh filename=package://unitree_go2_description/meshes/thigh.dae scale=1 1 1
- link lidar_l1_link: geometry collision mesh filename=package://unitree_go2_description/meshes/L1_4D_Lidar.dae scale=1 1 1; visual mesh filename=package://unitree_go2_description/meshes/L1_4D_Lidar.dae scale=1 1 1
- link rf_hip_link: geometry collision cylinder length=0.04 radius=0.046; visual mesh filename=package://unitree_go2_description/meshes/hip.dae scale=1 1 1
- link rf_lower_leg_link: geometry collision box size=0.213 0.016 0.016; visual mesh filename=package://unitree_go2_description/meshes/calf.dae scale=1 1 1
- link rf_upper_leg_link: geometry collision box size=0.213 0.0245 0.034; visual mesh filename=package://unitree_go2_description/meshes/thigh_mirror.dae scale=1 1 1
- link rh_hip_link: geometry collision cylinder length=0.04 radius=0.046; visual mesh filename=package://unitree_go2_description/meshes/hip.dae scale=1 1 1
- link rh_lower_leg_link: geometry collision box size=0.213 0.016 0.016; visual mesh filename=package://unitree_go2_description/meshes/calf.dae scale=1 1 1
- link rh_upper_leg_link: geometry collision box size=0.213 0.0245 0.034; visual mesh filename=package://unitree_go2_description/meshes/thigh_mirror.dae scale=1 1 1
- link trunk: geometry collision box size=0.3762 0.0935 0.114; visual mesh filename=package://unitree_go2_description/meshes/trunk.dae scale=1 1 1
- link velodyne: geometry visual mesh filename=package://unitree_go2_description/meshes/VLP16_scan.dae
- link velodyne_base_link: geometry collision cylinder length=0.0717 radius=0.0516; visual mesh filename=package://unitree_go2_description/meshes/VLP16_base_1.dae

Commit message: add a combined robot urdf

File: resource/go2.urdf (robot description, URDF)
Before this commit: robot go2, 23 links, 22 joints
Links:
- added link dummy_mimic_fix
- added link end_effector_link; visual box size=0.01 0.01 0.01
- added link gripper_left_link, mass 1.0e-03; collision mesh filename=package://webots_go2/protos/Omx/meshes/gripper_left_palm.stl scale=0.001 0.001 0.001; visual mesh filename=package://webots_go2/protos/Omx/meshes/gripper_left_palm.stl scale=0.001 0.001 0.001
- added link gripper_right_link, mass 1.0e-03; collision mesh filename=package://webots_go2/protos/Omx/meshes/gripper_right_palm.s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 scale=0.001 0.001 0.001; visual mesh filename=package://webots_go2/protos/Omx/meshes/gripper_right_palm.s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 scale=0.001 0.001 0.001
- added link link1, mass 7.9119962e-02; collision mesh filename=package://webots_go2/protos/Omx/meshes/link1.stl scale=0.001 0.001 0.001; visual mesh filename=package://webots_go2/protos/Omx/meshes/link1.stl scale=0.001 0.001 0.001
- added link link2, mass 9.8406837e-02; collision mesh filename=package://webots_go2/protos/Omx/meshes/link2.stl scale=0.001 0.001 0.001; visual mesh filename=package://webots_go2/protos/Omx/meshes/link2.stl scale=0.001 0.001 0.001
- added link link3, mass 1.3850917e-01; collision mesh filename=package://webots_go2/protos/Omx/meshes/link3.stl scale=0.001 0.001 0.001; visual mesh filename=package://webots_go2/protos/Omx/meshes/link3.stl scale=0.001 0.001 0.001
- added link link4, mass 1.3274562e-01; collision mesh filename=package://webots_go2/protos/Omx/meshes/link4.stl scale=0.001 0.001 0.001; visual mesh filename=package://webots_go2/protos/Omx/meshes/link4.stl scale=0.001 0.001 0.001
- added link link5, mass 1.4327573e-01; collision mesh filename=package://webots_go2/protos/Omx/meshes/link5.stl scale=0.001 0.001 0.001; visual mesh filename=package://webots_go2/protos/Omx/meshes/link5.stl scale=0.001 0.001 0.001
- link lf_hip_link: geometry collision cylinder length=0.04 radius=0.046; visual mesh filename=package://webots_go2/protos/Go2/meshes/hip.dae scale=1 1 1
- link lf_lower_leg_link: geometry collision box size=0.213 0.016 0.016; visual mesh filename=package://webots_go2/protos/Go2/meshes/calf.dae scale=1 1 1
- link lf_upper_leg_link: geometry collision box size=0.213 0.0245 0.034; visual mesh filename=package://webots_go2/protos/Go2/meshes/thigh.dae scale=1 1 1
- link lh_hip_link: geometry collision cylinder length=0.04 radius=0.046; visual mesh filename=package://webots_go2/protos/Go2/meshes/hip.dae scale=1 1 1
- link lh_lower_leg_link: geometry collision box size=0.213 0.016 0.016; visual mesh filename=package://webots_go2/protos/Go2/meshes/calf.dae scale=1 1 1
- link lh_upper_leg_link: geometry collision box size=0.213 0.0245 0.034; visual mesh filename=package://webots_go2/protos/Go2/meshes/thigh.dae scale=1 1 1
- link lidar_l1_link: geometry collision mesh filename=package://webots_go2/protos/Go2/meshes/L1_4D_Lidar.dae scale=1 1 1; visual mesh filename=package://webots_go2/protos/Go2/meshes/L1_4D_Lidar.dae scale=1 1 1
- link rf_hip_link: geometry collision cylinder length=0.04 radius=0.046; visual mesh filename=package://webots_go2/protos/Go2/meshes/hip.dae scale=1 1 1
- link rf_lower_leg_link: geometry collision box size=0.213 0.016 0.016; visual mesh filename=package://webots_go2/protos/Go2/meshes/calf.dae scale=1 1 1
- link rf_upper_leg_link: geometry collision box size=0.213 0.0245 0.034; visual mesh filename=package://webots_go2/protos/Go2/meshes/thigh_mirror.dae scale=1 1 1
- link rh_hip_link: geometry collision cylinder length=0.04 radius=0.046; visual mesh filename=package://webots_go2/protos/Go2/meshes/hip.dae scale=1 1 1
- link rh_lower_leg_link: geometry collision box size=0.213 0.016 0.016; visual mesh filename=package://webots_go2/protos/Go2/meshes/calf.dae scale=1 1 1
- link rh_upper_leg_link: geometry collision box size=0.213 0.0245 0.034; visual mesh filename=package://webots_go2/protos/Go2/meshes/thigh_mirror.dae scale=1 1 1
- link trunk: geometry collision box size=0.3762 0.0935 0.114; visual mesh filename=package://webots_go2/protos/Go2/meshes/trunk.dae scale=1 1 1
- link velodyne: geometry visual mesh filename=package://webots_go2/protos/Go2/meshes/VLP16_scan.dae
- link velodyne_base_link: geometry collision cylinder length=0.0717 radius=0.0516; visual mesh filename=package://webots_go2/protos/Go2/meshes/VLP16_base_1.dae
Joints:
- added joint end_effector_joint: type fixed, parent link5, child end_effector_link, origin xyz=0.126 0.0 0.0 rpy=0 0 0
- added joint go2_omx: type fixed, parent base_link, child link1, origin xyz=0.2 0 0.07 rpy=0 0 0
- added joint gripper_left_joint: type prismatic, parent link5, child gripper_left_link, origin xyz=0.0817 0.021 0.0 rpy=0 0 0, axis 0 1 0, limit lower=-0.010 upper=0.019 effort=1 velocity=4.8
- added joint gripper_right_joint: type prismatic, parent link5, child gripper_right_link, origin xyz=0.0817 -0.021 0 rpy=0 0 0, axis 0 -1 0, limit lower=-0.010 upper=0.019 effort=1 velocity=4.8, mimic joint=gripper_left_joint multiplier=1
- added joint gripper_right_joint_mimic: type fixed, parent gripper_right_link, child dummy_mimic_fix
- added joint joint1: type revolute, parent link1, child link2, origin xyz=0.012 0.0 0.017 rpy=0 0 0, axis 0 0 1, limit lower=-3.141592653589793 upper=3.141592653589793 effort=1 velocity=4.8
- added joint joint2: type revolute, parent link2, child link3, origin xyz=0.0 0.0 0.0595 rpy=0 0 0, axis 0 1 0, limit lower=-1.5 upper=1.5 effort=1 velocity=4.8
- added joint joint3: type revolute, parent link3, child link4, origin xyz=0.024 0 0.128 rpy=0 0 0, axis 0 1 0, limit lower=-1.5 upper=1.4 effort=1 velocity=4.8
- added joint joint4: type revolute, parent link4, child link5, origin xyz=0.124 0.0 0.0 rpy=0 0 0, axis 0 1 0, limit lower=-1.7 upper=1.97 effort=1 velocity=4.8
- joint velodyne_base_mount_joint: origin xyz=0.2 0 0.08 rpy=0 0 0 -> xyz=0 0 0.09 rpy=0 0 0

Commit message: Refactor robot from Spot to Go2
- Updated joint names and constraints in MoveGroupActionClient for new robot configuration.
- Changed launch file references from spot_launch.py to go2_launch.py.
- Modified joint state message handling to reflect new joint naming.
- Removed unused MoveGroupActionClient code in test_webots_nav2.py.
- Adjusted robot references in arena_modifier.py and retract_manipulator.py to Go2.
- Updated driver and service topics in spot_driver.py to align with Go2.
- Changed robot definition in go2.wbt to reflect new naming convention.
- Added new MoveIt SRDF file for Go2 robot configuration.

File: resource/go2.urdf (robot description, URDF)
Before this commit: robot go2, 32 links, 31 joints
Links:
- added link Velodyne_Puck
Joints:
- added joint velodyne_base_VelodynePuck: type fixed, parent velodyne, child Velodyne_Puck, origin xyz=0 0 0 rpy=0 0 0
